File: Hardware/COMPONENT_SHEETS/BAROMETER_MS5607-02.kicad_sch (KiCad schematic)
At the start: 2 parts, among them U1 MS5607-02BA

Commit message: Added correct crystal for mcu, re-routing of data lines in progress
Parts:
- renumbered C6 to C5
Other:
- note added: "Pressure range should be sufficient for ~100,000 feet."
- note removed: "MS5607-02 I2C Addresses: AD0 = 0 -> 0x77 AD0 = 1 -> 0x76"
- note removed: "Pressure range should be sufficientfor ~{} 100,000 feet."
Changed lines of the file:
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@@
     (stroke (width 0) (type default) (color 0 0 0 0))
   )
-  (text "Pressure range should be \nsufficientfor ~{} 100,000 feet."
+  (text "Pressure range should be \nsufficient for ~100,000 feet."
     (at 138.43 124.46 0)
-    (effects (font (size 1.27 1.27)) (justify left bottom))
-  )
-  (text "MS5607-02 I2C Addresses:\nAD0 = 0 -> 0x77\nAD0 = 1 -> 0x76"
-    (at 128.27 118.11 0)
     (effects (font (size 1.27 1.27)) (justify left bottom))
   )
@@
   (symbol (lib_id "power:+3.3V") (at 161.29 80.01 0) (unit 1)
     (in_bom yes) (on_board yes)
-    (property "Reference" "#PWR0101" (id 0) (at 161.29 83.82 0)
+    (property "Reference" "#PWR013" (id 0) (at 161.29 83.82 0)
       (effects (font (size 1.27 1.27)) hide)
     )
@@
     (pin "1")
   )
-  (symbol (lib_id "Device:C_Small") (at 161.29 91.44 180)
+  (symbol (lib_id "Device:C_Small") (at 161.29 91.44 180) (unit 1)
     (in_bom yes) (on_board yes)
-    (property "Reference" "C6" (id 0) (at 163.6268 90.2716 0)
+    (property "Reference" "C5" (id 0) (at 163.6268 90.2716 0)
       (effects (font (size 1.27 1.27)) (justify right))
     )
@@
   (symbol (lib_id "power:GND") (at 149.86 105.41 0) (unit 1)
     (in_bom yes) (on_board yes)
-    (property "Reference" "#PWR0102" (id 0) (at 149.86 111.76 0)
+    (property "Reference" "#PWR012" (id 0) (at 149.86 111.76 0)
       (effects (font (size 1.27 1.27)) hide)
     )
