File: Hardware/COMPONENT_SHEETS/STM32L562VET6Q.kicad_sch (KiCad schematic)
At the start: 7 parts, among them IC2 STM32L562VET6Q, Y1 32mhz

Commit message: Added correct crystal for mcu, re-routing of data lines in progress
Connections:
- net Buzzer_Excitation: no longer names the net of IC2.31 (PA7)
- net Fire_A: no longer names the net of IC2.60 (PD13)
- net Fire_B: no longer names the net of IC2.59 (PD12)
- net Fire_C: no longer names the net of IC2.56 (PD9)
- net Fire_D: no longer names the net of IC2.55 (PD8)
- net Sense_A: no longer names the net of IC2.58 (PD11)
- net Sense_B: no longer names the net of IC2.61 (PD14)
- net Sense_C: no longer names the net of IC2.54 (PB15)
- net Sense_D: no longer names the net of IC2.57 (PD10)
Changed lines of the file:
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@@
-    (effects (font (size 1.27 1.27)) (justify left))
-  )
-  (hierarchical_label "Sense_B" (shape input) (at 168.91 91.44 0)
-    (effects (font (size 1.27 1.27)) (justify left))
-  )
-  (hierarchical_label "Fire_A" (shape input) (at 168.91 93.98 0)
-    (effects (font (size 1.27 1.27)) (justify left))
-  )
-  (hierarchical_label "Fire_C" (shape input) (at 168.91 104.14 0)
-    (effects (font (size 1.27 1.27)) (justify left))
-  )
-  (hierarchical_label "Sense_D" (shape input) (at 168.91 101.6 0)
-    (effects (font (size 1.27 1.27)) (justify left))
-  )
-  (hierarchical_label "Sense_C" (shape input) (at 168.91 109.22 0)
     (effects (font (size 1.27 1.27)) (justify left))
   )
@@
     (effects (font (size 1.27 1.27)) (justify right))
   )
-  (hierarchical_label "Sense_A" (shape input) (at 168.91 99.06 0)
-    (effects (font (size 1.27 1.27)) (justify left))
-  )
-  (hierarchical_label "Buzzer_Excitation" (shape input) (at 113.03 139.7 270)
-    (effects (font (size 1.27 1.27)) (justify right))
-  )
   (hierarchical_label "SWCLK" (shape input) (at 158.75 33.02 90)
     (effects (font (size 1.27 1.27)) (justify left))
@@
     (effects (font (size 1.27 1.27)) (justify left))
   )
-  (hierarchical_label "Fire_B" (shape input) (at 168.91 96.52 0)
-    (effects (font (size 1.27 1.27)) (justify left))
-  )
   (hierarchical_label "I2C1_SCL" (shape input) (at 156.21 33.02 90)
     (effects (font (size 1.27 1.27)) (justify left))
   )
-  (hierarchical_label "Fire_D" (shape input) (at 168.91 106.68 0)
-    (effects (font (size 1.27 1.27)) (justify left))
-  )
